Commit message: fixed the warning about world and base_link.

File: urdf_tutorial/urdf/roboturdf.urdf (robot description, URDF)
Before this commit: robot roboturdf, 7 links, 6 joints
Links:
- added link world_link
Joints:
- added joint world_fixed_joint: type fixed, parent world_link, child base_link, origin xyz=0 0 0 rpy=0 0 0
